Commit message: Add gazebo simulation

File: ur5e_moveit_config/urdf/panther_base_macro.urdf.xacro (robot description, xacro)
@@ -15,4 +15,5 @@
     <xacro:include filename="$(find panther_description)/urdf/body.urdf.xacro" ns="body" />
     <xacro:include filename="$(find panther_description)/urdf/wheel.urdf.xacro" ns="wheel" />
+    <xacro:include filename="$(find panther_description)/urdf/gazebo_plugins.gazebo.xacro" ns="gazebo" />
     <!-- BODY DECLARATION -->
     <xacro:body.body props="${panther_common_props['body']}" wheel_props="${wheel_props['wheels']}" />
@@ -22,4 +23,5 @@
     <xacro:wheel.wheel wheel_props="${wheel_props['wheels']}" common_props="${panther_common_props}" prefix="rear_left" />
     <xacro:wheel.wheel wheel_props="${wheel_props['wheels']}" common_props="${panther_common_props}" prefix="rear_right" />
+    <xacro:gazebo.wheel_driver wheel_props="${wheel_props}" common_props="${panther_common_props}" />
   </xacro:macro>
 </robot>

File: ur5e_moveit_config/urdf/power_supply_macro.xacro (robot description, xacro)
@@ -17,10 +17,7 @@
       </visual>
       <inertial>
-        <origin xyz="0 0 1" rpy="0 0 0"/>
-        <mass value="1"/>
-        <inertia
-          ixx="1.0" ixy="0.0" ixz="0.0"
-          iyy="1.0" iyz="0.0"
-          izz="1.0"/>
+        <mass value="0.59" />
+        <inertia ixx="0.003964" ixy="0.0" ixz="0.0" iyy="0.0003964" iyz="0.0" izz="0.0004177" />
+        <origin xyz="0.045 0.0 0.0058" rpy="0.0 0.0 0.0"/>
       </inertial>
     </link>

File: ur5e_moveit_config/urdf/ur_macro.xacro (robot description, xacro)
@@ -316,4 +316,36 @@
       <child link="${prefix}tool0"/>
     </joint>
+    <!-- Configure self collision properties per link -->
+    <gazebo reference="${prefix}shoulder_link">
+      <selfCollide>true</selfCollide>
+    </gazebo>
+    <gazebo reference="${prefix}upper_arm_link">
+      <selfCollide>true</selfCollide>
+    </gazebo>
+    <gazebo reference="${prefix}forearm_link">
+      <selfCollide>true</selfCollide>
+    </gazebo>
+    <gazebo reference="${prefix}wrist_1_link">
+      <selfCollide>true</selfCollide>
+    </gazebo>
+    <gazebo reference="${prefix}wrist_3_link">
+      <selfCollide>true</selfCollide>
+    </gazebo>
+    <gazebo reference="${prefix}wrist_2_link">
+      <selfCollide>true</selfCollide>
+    </gazebo>
+    <gazebo reference="${prefix}ee_link">
+      <selfCollide>true</selfCollide>
+    </gazebo>
+    <!--
+      Inject Gazebo ROS Control plugin, which allows us to use ros_control
+      controllers to control the virtual robot hw.
+    -->
+    <gazebo>
+      <plugin name="ros_control" filename="libgazebo_ros_control.so">
+        <!--robotNamespace>/</robotNamespace-->
+        <!--robotSimType>gazebo_ros_control/DefaultRobotHWSim</robotSimType-->
+      </plugin>
+    </gazebo>
   </xacro:macro>
 </robot>
