Commit message: Fix review comments || Add upper rails

File: ur5e_moveit_config/urdf/external_antena_macro.urdf.xacro (robot description, xacro)
@@ -26,5 +26,5 @@
           <mesh filename="file://$(find ur5e_moveit_config)/meshes/external_antenna.dae" />
         </geometry>
-        <origin xyz="0.0 0.0 0.0" rpy="0.0 0.0 0.0"/>
+        <origin xyz="0.0 0.0 0.0" rpy="0.0 0.0 0.0" />
       </visual>
       <collision>
@@ -32,10 +32,10 @@
           <mesh filename="file://$(find ur5e_moveit_config)/meshes/external_antenna_collision.stl" />
         </geometry>
-        <origin xyz="0.0 0.0 0.0" rpy="0.0 0.0 0.0"/>
+        <origin xyz="0.0 0.0 0.0" rpy="0.0 0.0 0.0" />
       </collision>
       <inertial>
         <mass value="0.59" />
         <inertia ixx="0.003964" ixy="0.0" ixz="0.0" iyy="0.0003964" iyz="0.0" izz="0.0004177" />
-        <origin xyz="0.045 0.0 0.0058" rpy="0.0 0.0 0.0"/>
+        <origin xyz="0.045 0.0 0.0058" rpy="0.0 0.0 0.0" />
       </inertial>
     </link>

File: ur5e_moveit_config/urdf/panther_base_macro.urdf.xacro (robot description, xacro)
@@ -7,7 +7,7 @@
     <xacro:arg name="use_gpu" default="false" />
     <!-- IMPORT YAML CONFIGS -->
-    <xacro:property name="panther_common_props_file" value="$(arg panther_common_props_path)"  />
+    <xacro:property name="panther_common_props_file" value="$(arg panther_common_props_path)" />
     <xacro:property name="panther_common_props" value="${xacro.load_yaml(panther_common_props_file)}" />
-    <xacro:property name="wheel_props_file" value="$(arg wheel_props_path)"  />
+    <xacro:property name="wheel_props_file" value="$(arg wheel_props_path)" />
     <xacro:property name="wheel_props" value="${xacro.load_yaml(wheel_props_file)}" />
     <!-- INCLUDE ROBOT PARTS DEFINITIONS -->

File: ur5e_moveit_config/urdf/panther_ur5e.urdf.xacro (robot description, xacro)
@@ -10,12 +10,12 @@
           when updating the package to the latest version of panther_description,
           add rails that reflect the actual components -->
-  <!-- <xacro:include filename="$(find ur5e_moveit_config)/urdf/upper_rails.urdf.xacro" ns="rails" /> -->
-  <!-- <xacro:rails.upper_rails parent_link="base_link" xyz="0.0 0.0 0.334" rpy="0.0 ${-pi/2} 0.0"  /> -->
+  <xacro:include filename="$(find ur5e_moveit_config)/urdf/upper_rails.urdf.xacro" ns="rails" />
+  <xacro:rails.upper_rails parent_link="base_link" xyz="0.0 0.0 0.334" rpy="0.0 ${-pi/2} 0.0" />
   <xacro:husarion.panther_base  />
-  <xacro:antena.external_antenna parent_link="base_link" xyz="0.18 0.15 0.377" rpy="0.0 0.0 ${pi}"  />
-  <xacro:power_supply.power_supply parent_link="base_link" xyz="0.0 -0.13 0.377" rpy="0.0 0.0 0.0"  />
+  <xacro:antena.external_antenna parent_link="base_link" xyz="0.18 0.15 0.377" rpy="0.0 0.0 ${pi}" />
+  <xacro:power_supply.power_supply parent_link="base_link" xyz="0.0 -0.13 0.377" rpy="0.0 0.0 0.0" />
   <xacro:velodyne.velodyne_puck parent_link="base_link" xyz="0.05 -0.13 0.527" rpy="0.0 0.0 0.0" />
   <xacro:rs.sensor_d435i parent="base_link" use_nominal_extrinsics="true">
-    <origin xyz="0.19 0.05 0.427" rpy="0 0 0"/>
+    <origin xyz="0.19 0.05 0.427" rpy="0 0 0" />
   </xacro:rs.sensor_d435i>
   <xacro:universal_robot.ur_robot

File: ur5e_moveit_config/urdf/power_supply_macro.xacro (robot description, xacro)
@@ -5,5 +5,5 @@
     <link name="power_supply_link">
       <collision>
-        <origin xyz="0.0 0.09 0.15" rpy="${-pi/2} 0 ${pi}"/>
+        <origin xyz="0.0 0.09 0.15" rpy="${-pi/2} 0.0 ${pi}"/>
         <geometry>
           <mesh filename="file://$(find ur5e_moveit_config)/meshes/power_supply.stl" scale="0.011 0.011 0.011" />
@@ -11,5 +11,5 @@
       </collision>
       <visual>
-        <origin xyz="0.0 0.09 0.15" rpy="${-pi/2} 0 ${pi}"/>
+        <origin xyz="0.0 0.09 0.15" rpy="${-pi/2} 0.0 ${pi}"/>
         <geometry>
           <mesh filename="file://$(find ur5e_moveit_config)/meshes/power_supply.dae" scale="0.01 0.01 0.01" />
@@ -19,5 +19,5 @@
         <mass value="0.59" />
         <inertia ixx="0.003964" ixy="0.0" ixz="0.0" iyy="0.0003964" iyz="0.0" izz="0.0004177" />
-        <origin xyz="0.045 0.0 0.0058" rpy="0.0 0.0 0.0"/>
+        <origin xyz="0.045 0.0 0.0058" rpy="0.0 0.0 0.0" />
       </inertial>
     </link>

File: ur5e_moveit_config/urdf/upper_rails.urdf.xacro (robot description, xacro)
@@ -8,5 +8,5 @@
           <mesh filename="file://$(find ur5e_moveit_config)/meshes/upper_rails.stl" scale="0.01 0.01 0.01" />
         </geometry>
-        <origin xyz="0 0 0" rpy=" ${pi/2} 0 ${pi/2}"/>
+        <origin xyz="0.0 0.0 0.0" rpy=" ${pi/2} 0.0 ${pi/2}" />
       </collision>
       <visual>
@@ -14,10 +14,10 @@
           <mesh filename="file://$(find ur5e_moveit_config)/meshes/upper_rails.stl" scale="0.01 0.01 0.01" />
         </geometry>
-        <origin xyz="0 0 0" rpy=" ${pi/2} 0 ${pi/2}"/>
-        <material name="Black"/>
+        <origin xyz="0.0 0.0 0.0" rpy=" ${pi/2} 0.0 ${pi/2}" />
+        <material name="Black" />
       </visual>
       <inertial>
         <mass value="0.0000001" />
-        <inertia ixx="1" ixy="0" ixz="0" iyy="1" iyz="0" izz="1" />
+        <inertia ixx="1.0" ixy="0.0" ixz="0.0" iyy="1.0" iyz="0.0" izz="1.0" />
       </inertial>
     </link>
@@ -27,4 +27,7 @@
       <child link="upper_rails_link" />
     </joint>
+    <gazebo reference="upper_rails_link">
+      <material>Gazebo/Black</material>
+    </gazebo>
   </xacro:macro>
 </robot>
