Commit message: Update ur5e_moveit_config/urdf/power_supply_macro.xacro
Co-authored-by: Dawid Kmak <73443304+KmakD@users.noreply.github.com>

File: ur5e_moveit_config/urdf/power_supply_macro.xacro (robot description, xacro)
@@ -5,5 +5,5 @@
     <link name="power_supply_link">
       <collision>
-        <origin xyz="0.0 0.09 0.15" rpy="${-pi/2} 0.0 ${pi}"/>
+        <origin xyz="0.0 0.09 0.15" rpy="${-pi/2} 0.0 ${pi}" />
         <geometry>
           <mesh filename="file://$(find ur5e_moveit_config)/meshes/power_supply.stl" scale="0.011 0.011 0.011" />

Commit message: Update ur5e_moveit_config/urdf/power_supply_macro.xacro
Co-authored-by: Dawid Kmak <73443304+KmakD@users.noreply.github.com>

File: ur5e_moveit_config/urdf/power_supply_macro.xacro (robot description, xacro)
@@ -11,5 +11,5 @@
       </collision>
       <visual>
-        <origin xyz="0.0 0.09 0.15" rpy="${-pi/2} 0.0 ${pi}"/>
+        <origin xyz="0.0 0.09 0.15" rpy="${-pi/2} 0.0 ${pi}" />
         <geometry>
           <mesh filename="file://$(find ur5e_moveit_config)/meshes/power_supply.dae" scale="0.01 0.01 0.01" />
