Commit message: update urdf

File: ur5e_moveit_config/urdf/panther_ur5e.urdf.xacro (robot description, xacro)
@@ -3,11 +3,17 @@
   <xacro:include filename="$(find ur5e_moveit_config)/urdf/panther_base_macro.urdf.xacro" ns="husarion" />
   <xacro:include filename="$(find ur5e_moveit_config)/urdf/ur_macro.xacro" ns="universal_robot"/>
+  <xacro:include filename="$(find ur5e_moveit_config)/urdf/upper_rails.urdf.xacro" ns="rails" />
   <xacro:include filename="$(find ur5e_moveit_config)/urdf/external_antena_macro.urdf.xacro" ns="antena" />
   <xacro:include filename="$(find ur5e_moveit_config)/urdf/power_supply_macro.xacro" ns="power_supply"/>
   <xacro:include filename="$(find panther_description)/urdf/components/velodyne_puck.gazebo.xacro" ns="velodyne" />
+  <xacro:include filename="$(find realsense2_description)/urdf/_d435i.urdf.xacro" ns="rs"/>
   <xacro:husarion.panther_base  />
-  <xacro:antena.external_antenna parent_link="base_link" xyz="0.18 0.15 0.377" rpy="0 0 3.1415"  />
-  <xacro:power_supply.power_supply parent_link="base_link" xyz="0.0 -0.065 0.227" rpy="0 0 0.0"  />
-  <xacro:velodyne.velodyne_puck xyz="0.05 -0.13 0.357" rpy="0 0 0" />
+  <xacro:rails.upper_rails parent_link="base_link" xyz="0.0 0.0 0.334" rpy="0.0 ${-pi/2} 0.0"  />
+  <xacro:antena.external_antenna parent_link="base_link" xyz="0.18 0.15 0.377" rpy="0.0 0.0 ${pi}"  />
+  <xacro:power_supply.power_supply parent_link="base_link" xyz="0.0 -0.13 0.377" rpy="0.0 0.0 0.0"  />
+  <xacro:velodyne.velodyne_puck xyz="0.05 -0.13 0.35" rpy="0.0 0.0 0.0" />
+  <xacro:rs.sensor_d435i parent="base_link" use_nominal_extrinsics="true">
+    <origin xyz="0.19 0.05 0.427" rpy="0 0 0"/>
+  </xacro:rs.sensor_d435i>
   <xacro:universal_robot.ur_robot
     prefix=""
@@ -22,5 +28,5 @@
   />
   <joint name="base_link_to_ur5e_link_joint" type="fixed">
-    <origin xyz="-0.10 0.10 0.375" rpy="0 0 1.54" />
+    <origin xyz="-0.095 0.0975 0.375" rpy="0 0 ${pi/2}" />
     <parent link="base_link" />
     <child link="ur5e_link" />

File: ur5e_moveit_config/urdf/power_supply_macro.xacro (robot description, xacro)
@@ -5,13 +5,13 @@
     <link name="power_supply_link">
       <collision>
-        <origin xyz="${xyz}" rpy="${rpy}"/>
+        <origin xyz="0.0 0.09 0.15" rpy="${-pi/2} 0 ${pi}"/>
         <geometry>
-          <box size="0.57 0.26 0.15"/>
+          <mesh filename="file://$(find ur5e_moveit_config)/meshes/power_supply.stl" scale="0.011 0.011 0.011" />
         </geometry>
       </collision>
       <visual>
-        <origin xyz="${xyz}" rpy="${rpy}"/>
+        <origin xyz="0.0 0.09 0.15" rpy="${-pi/2} 0 ${pi}"/>
         <geometry>
-          <box size="0.57 0.26 0.15"/>
+          <mesh filename="file://$(find ur5e_moveit_config)/meshes/power_supply.dae" scale="0.01 0.01 0.01" />
         </geometry>
       </visual>
@@ -30,7 +30,4 @@
       <child link="power_supply_link" />
     </joint>
-    <gazebo reference="power_supply_link">
-      <material>Gazebo/DarkGrey</material>
-    </gazebo>
   </xacro:macro>
 </robot>

Commit message: fix rviz model || code cleanup

File: ur5e_moveit_config/urdf/panther_ur5e.urdf.xacro (robot description, xacro)
@@ -3,11 +3,14 @@
   <xacro:include filename="$(find ur5e_moveit_config)/urdf/panther_base_macro.urdf.xacro" ns="husarion" />
   <xacro:include filename="$(find ur5e_moveit_config)/urdf/ur_macro.xacro" ns="universal_robot"/>
-  <xacro:include filename="$(find ur5e_moveit_config)/urdf/upper_rails.urdf.xacro" ns="rails" />
   <xacro:include filename="$(find ur5e_moveit_config)/urdf/external_antena_macro.urdf.xacro" ns="antena" />
   <xacro:include filename="$(find ur5e_moveit_config)/urdf/power_supply_macro.xacro" ns="power_supply"/>
   <xacro:include filename="$(find panther_description)/urdf/components/velodyne_puck.gazebo.xacro" ns="velodyne" />
   <xacro:include filename="$(find realsense2_description)/urdf/_d435i.urdf.xacro" ns="rs"/>
+  <!-- !TODO:
+          when updating the package to the latest version of panther_description,
+          add rails that reflect the actual components -->
+  <!-- <xacro:include filename="$(find ur5e_moveit_config)/urdf/upper_rails.urdf.xacro" ns="rails" /> -->
+  <!-- <xacro:rails.upper_rails parent_link="base_link" xyz="0.0 0.0 0.334" rpy="0.0 ${-pi/2} 0.0"  /> -->
   <xacro:husarion.panther_base  />
-  <xacro:rails.upper_rails parent_link="base_link" xyz="0.0 0.0 0.334" rpy="0.0 ${-pi/2} 0.0"  />
   <xacro:antena.external_antenna parent_link="base_link" xyz="0.18 0.15 0.377" rpy="0.0 0.0 ${pi}"  />
   <xacro:power_supply.power_supply parent_link="base_link" xyz="0.0 -0.13 0.377" rpy="0.0 0.0 0.0"  />

File: ur5e_moveit_config/urdf/upper_rails.urdf.xacro (robot description, xacro)
@@ -4,8 +4,10 @@
               params="parent_link xyz rpy">
     <link name="upper_rails_link">
-      <inertial>
-        <mass value="0.0000001" />
-        <inertia ixx="1" ixy="0" ixz="0" iyy="1" iyz="0" izz="1" />
-      </inertial>
+      <collision>
+        <geometry>
+          <mesh filename="file://$(find ur5e_moveit_config)/meshes/upper_rails.stl" scale="0.01 0.01 0.01" />
+        </geometry>
+        <origin xyz="0 0 0" rpy=" ${pi/2} 0 ${pi/2}"/>
+      </collision>
       <visual>
         <geometry>
@@ -15,4 +17,8 @@
         <material name="Black"/>
       </visual>
+      <inertial>
+        <mass value="0.0000001" />
+        <inertia ixx="1" ixy="0" ixz="0" iyy="1" iyz="0" izz="1" />
+      </inertial>
     </link>
     <joint name="${parent_link}_to_upper_rails_link_joint" type="fixed">

Commit message: Update ur5e_moveit_config/urdf/panther_ur5e.urdf.xacro
Co-authored-by: Dawid Kmak <73443304+KmakD@users.noreply.github.com>

File: ur5e_moveit_config/urdf/panther_ur5e.urdf.xacro (robot description, xacro)
@@ -17,5 +17,5 @@
   <xacro:velodyne.velodyne_puck parent_link="base_link" xyz="0.05 -0.13 0.527" rpy="0.0 0.0 0.0" />
   <xacro:rs.sensor_d435i parent="base_link" use_nominal_extrinsics="true">
-    <origin xyz="0.19 0.05 0.427" rpy="0 0 0" />
+    <origin xyz="0.19 0.05 0.427" rpy="0.0 0.0 0.0" />
   </xacro:rs.sensor_d435i>
   <xacro:universal_robot.ur_robot

Commit message: Update ur5e_moveit_config/urdf/panther_ur5e.urdf.xacro
Co-authored-by: Dawid Kmak <73443304+KmakD@users.noreply.github.com>

File: ur5e_moveit_config/urdf/panther_ur5e.urdf.xacro (robot description, xacro)
@@ -31,5 +31,5 @@
   />
   <joint name="base_link_to_ur5e_link_joint" type="fixed">
-    <origin xyz="-0.095 0.0975 0.375" rpy="0 0 ${pi/2}" />
+    <origin xyz="-0.095 0.0975 0.375" rpy="0.0 0.0 ${pi/2}" />
     <parent link="base_link" />
     <child link="ur5e_link" />

Commit message: add ur3 gazebo sim

File: ur5e_moveit_config/urdf/panther_ur5e.urdf.xacro (robot description, xacro)
@@ -7,7 +7,5 @@
   <xacro:include filename="$(find panther_description)/urdf/panther_macro.urdf.xacro" ns="husarion" />
   <xacro:include filename="$(find ur_description)/urdf/inc/ur5e_macro.xacro" ns="universal_robot"/>
-  <xacro:husarion.panther_robot
-    dual_bat="$(arg dual_bat)"
-    wheel_config_path="$(arg wheel_config_path)" />
+  <xacro:husarion.panther_robot dual_bat="$(arg dual_bat)" wheel_config_path="$(arg wheel_config_path)" />
   <xacro:universal_robot.ur5e_robot prefix="panther_ur5e_" />
   <joint name="base_link_to_ur5e_link_joint" type="fixed">
@@ -25,6 +23,6 @@
   <!-- Components -->
   <xacro:include filename="$(find panther_description)/urdf/components/external_antenna.urdf.xacro" ns="antena" />
-  <xacro:include filename="$(find ur5e_components_description)/urdf/power_supply.urdf.xacro" ns="power_supply" />
-  <xacro:include filename="$(find ur5e_components_description)/urdf/upper_rails.urdf.xacro" ns="rails" />
+  <xacro:include filename="$(find ur_components_description)/urdf/power_supply.urdf.xacro" ns="power_supply" />
+  <xacro:include filename="$(find ur_components_description)/urdf/upper_rails.urdf.xacro" ns="rails" />
   <xacro:antena.external_antenna parent_link="base_link" xyz="0.18 0.15 0.377" rpy="0.0 0.0 ${pi}" />
   <xacro:power_supply.power_supply parent_link="base_link" xyz="0.0 -0.13 0.377" rpy="0.0 0.0 0.0" />

File: ur_components_description/urdf/power_supply.urdf.xacro (robot description, xacro)
@@ -7,5 +7,5 @@
         <origin xyz="0.0 0.09 0.15" rpy="${-pi/2} 0.0 ${pi}" />
         <geometry>
-          <mesh filename="file://$(find ur5e_components_description)/meshes/power_supply.stl" scale="0.011 0.011 0.011" />
+          <mesh filename="file://$(find ur_components_description)/meshes/power_supply.stl" scale="0.011 0.011 0.011" />
         </geometry>
       </collision>
@@ -13,5 +13,5 @@
         <origin xyz="0.0 0.09 0.15" rpy="${-pi/2} 0.0 ${pi}" />
         <geometry>
-          <mesh filename="file://$(find ur5e_components_description)/meshes/power_supply.dae" scale="0.01 0.01 0.01" />
+          <mesh filename="file://$(find ur_components_description)/meshes/power_supply.dae" scale="0.01 0.01 0.01" />
         </geometry>
       </visual>

File: ur_components_description/urdf/upper_rails.urdf.xacro (robot description, xacro)
@@ -6,5 +6,5 @@
       <collision>
         <geometry>
-          <mesh filename="file://$(find ur5e_components_description)/meshes/upper_rails.stl" scale="0.01 0.01 0.01" />
+          <mesh filename="file://$(find ur_components_description)/meshes/upper_rails.stl" scale="0.01 0.01 0.01" />
         </geometry>
         <origin xyz="0.0 0.0 0.0" rpy=" ${pi/2} 0.0 ${pi/2}" />
@@ -12,5 +12,5 @@
       <visual>
         <geometry>
-          <mesh filename="file://$(find ur5e_components_description)/meshes/upper_rails.stl" scale="0.01 0.01 0.01" />
+          <mesh filename="file://$(find ur_components_description)/meshes/upper_rails.stl" scale="0.01 0.01 0.01" />
         </geometry>
         <origin xyz="0.0 0.0 0.0" rpy=" ${pi/2} 0.0 ${pi/2}" />

Commit message: gripper - add ros-control

File: ur5e_moveit_config/urdf/panther_ur5e.urdf.xacro (robot description, xacro)
@@ -5,8 +5,10 @@
   <xacro:arg name="wheel_config_path" default="$(find panther_description)/config/WH01.yaml" />
   <!-- Robot -->
-  <!-- <xacro:include filename="$(find ur5e_moveit_config)/urdf/panther_temp_macro.urdf.xacro" ns="husarion" /> -->
   <xacro:include filename="$(find panther_description)/urdf/panther_macro.urdf.xacro" ns="husarion" />
-  <xacro:include filename="$(find ur_description)/urdf/inc/ur5e_macro.xacro" ns="universal_robot"/>
-  <xacro:husarion.panther_robot dual_bat="$(arg dual_bat)" wheel_config_path="$(arg wheel_config_path)" />
+  <xacro:include filename="$(find ur_description)/urdf/inc/ur5e_macro.xacro" ns="universal_robot" />
+  <xacro:husarion.panther_robot
+    dual_bat="$(arg dual_bat)"
+    wheel_config_path="$(arg wheel_config_path)"
+    use_ros_control="True" />
   <xacro:universal_robot.ur5e_robot prefix="panther_ur5e_" />
   <joint name="base_link_to_ur5e_link_joint" type="fixed">
@@ -16,13 +18,17 @@
   </joint>
   <!-- Sensors -->
-  <xacro:include filename="$(find ros_components_description)/urdf/velodyne_puck.urdf.xacro" ns="velodyne" />
+  <xacro:include filename="$(find ros_components_description)/urdf/velodyne_puck.urdf.xacro"
+    ns="velodyne" />
   <xacro:include filename="$(find realsense2_description)/urdf/_d435i.urdf.xacro" ns="rs" />
-  <xacro:velodyne.velodyne_puck parent_link="base_link" xyz="0.05 -0.13 0.527" rpy="0.0 0.0 0.0" use_gpu="$(arg use_gpu)" />
+  <xacro:velodyne.velodyne_puck parent_link="base_link" xyz="0.05 -0.13 0.527" rpy="0.0 0.0 0.0"
+    use_gpu="$(arg use_gpu)" />
   <xacro:rs.sensor_d435i parent="base_link" use_nominal_extrinsics="true">
     <origin xyz="0.19 0.05 0.427" rpy="0.0 0.0 0.0" />
   </xacro:rs.sensor_d435i>
   <!-- Components -->
-  <xacro:include filename="$(find panther_description)/urdf/components/external_antenna.urdf.xacro" ns="antena" />
-  <xacro:include filename="$(find ur_components_description)/urdf/power_supply.urdf.xacro" ns="power_supply" />
+  <xacro:include filename="$(find panther_description)/urdf/components/external_antenna.urdf.xacro"
+    ns="antena" />
+  <xacro:include filename="$(find ur_components_description)/urdf/power_supply.urdf.xacro"
+    ns="power_supply" />
   <xacro:include filename="$(find ur_components_description)/urdf/upper_rails.urdf.xacro" ns="rails" />
   <xacro:antena.external_antenna parent_link="base_link" xyz="0.18 0.15 0.377" rpy="0.0 0.0 ${pi}" />

File: ur5e_onrobot_rg2_moveit_config/urdf/panther_ur5e_rg2.urdf.xacro (robot description, xacro)
@@ -8,7 +8,10 @@
   <xacro:include filename="$(find ur_description)/urdf/inc/ur5e_macro.xacro" ns="universal_robot"/>
   <xacro:include filename="$(find ur_components_description)/urdf/onrobot_rg2.urdf.xacro" ns="onrobot" />
-  <xacro:husarion.panther_robot dual_bat="$(arg dual_bat)" wheel_config_path="$(arg wheel_config_path)" />
+  <xacro:husarion.panther_robot
+    dual_bat="$(arg dual_bat)"
+    wheel_config_path="$(arg wheel_config_path)"
+    use_ros_control="True" />
   <xacro:universal_robot.ur5e_robot prefix="panther_ur5e_" />
-  <xacro:onrobot.onrobot_rg2 parent_link="panther_ur5e_tool0" xyz="0.0 0.0 0.0" rpy="-1.54 -1.54 0.0" />
+  <xacro:onrobot.onrobot_rg2 parent_link="panther_ur5e_tool0" xyz="0.0 0.0 0.02" rpy="${-pi/2} ${-pi/2} 0.0" />
   <joint name="base_link_to_ur5e_link_joint" type="fixed">
     <origin xyz="-0.095 0.0975 0.375" rpy="0.0 0.0 ${pi/2}" />

File: ur_components_description/urdf/onrobot_rg2.urdf.xacro (robot description, xacro)
@@ -50,11 +50,11 @@
         <origin xyz="0.0 0.0 0.0" rpy="0.0 0.0 0.0" />
         <geometry>
-          <mesh filename="file://$(find ur_components_description)/meshes/onrobot/collision/RG2_Hand_col.STL" />
-        </geometry>
-      </collision>
-      <visual>
-        <origin xyz="0.0 0.0 0.0" rpy="0.0 0.0 0.0" />
-        <geometry>
-          <mesh filename="file://$(find ur_components_description)/meshes/onrobot/visual/RG2_Hand_vis.STL" />
+          <mesh filename="file://$(find ur_components_description)/meshes/onrobot/hand.stl" />
+        </geometry>
+      </collision>
+      <visual>
+        <origin xyz="0.0 0.0 0.0" rpy="0.0 0.0 0.0" />
+        <geometry>
+          <mesh filename="file://$(find ur_components_description)/meshes/onrobot/hand.dae" />
         </geometry>
       </visual>
@@ -81,11 +81,11 @@
         <origin xyz="0.0 0.0 0.0" rpy="0.0 0.0 0.0" />
         <geometry>
-          <mesh filename="file://$(find ur_components_description)/meshes/onrobot/collision/RG2_LeftMomentArm_col.STL" />
-        </geometry>
-      </collision>
-      <visual>
-        <origin xyz="0.0 0.0 0.0" rpy="0.0 0.0 0.0" />
-        <geometry>
-          <mesh filename="file://$(find ur_components_description)/meshes/onrobot/visual/RG2_LeftMomentArm_vis.STL" />
+          <mesh filename="file://$(find ur_components_description)/meshes/onrobot/moment_arm.stl" />
+        </geometry>
+      </collision>
+      <visual>
+        <origin xyz="0.0 0.0 0.0" rpy="0.0 0.0 0.0" />
+        <geometry>
+          <mesh filename="file://$(find ur_components_description)/meshes/onrobot/moment_arm.dae" />
         </geometry>
       </visual>
@@ -118,11 +118,11 @@
         <origin xyz="0.0 0.0 0.0" rpy="0.0 0.0 0.0" />
         <geometry>
-          <mesh filename="file://$(find ur_components_description)/meshes/onrobot/collision/RG2_LeftFinger_col.STL" />
-        </geometry>
-      </collision>
-      <visual>
-        <origin xyz="0.0 0.0 0.0" rpy="0.0 0.0 0.0" />
-        <geometry>
-          <mesh filename="file://$(find ur_components_description)/meshes/onrobot/visual/RG2_LeftFinger_vis.STL" />
+          <mesh filename="file://$(find ur_components_description)/meshes/onrobot/finger.stl" />
+        </geometry>
+      </collision>
+      <visual>
+        <origin xyz="0.0 0.0 0.0" rpy="0.0 0.0 0.0" />
+        <geometry>
+          <mesh filename="file://$(find ur_components_description)/meshes/onrobot/finger.dae" />
         </geometry>
       </visual>
@@ -155,11 +155,11 @@
         <origin xyz="0.0 0.0 0.0" rpy="0.0 0.0 0.0" />
         <geometry>
-          <mesh filename="file://$(find ur_components_description)/meshes/onrobot/collision/RG2_LeftTrussArm_col.STL" />
-        </geometry>
-      </collision>
-      <visual>
-        <origin xyz="0.0 0.0 0.0" rpy="0.0 0.0 0.0" />
-        <geometry>
-          <mesh filename="file://$(find ur_components_description)/meshes/onrobot/visual/RG2_LeftTrussArm_vis.STL" />
+          <mesh filename="file://$(find ur_components_description)/meshes/onrobot/truss_arm.stl" />
+        </geometry>
+      </collision>
+      <visual>
+        <origin xyz="0.0 0.0 0.0" rpy="0.0 0.0 0.0" />
+        <geometry>
+          <mesh filename="file://$(find ur_components_description)/meshes/onrobot/truss_arm.dae" />
         </geometry>
       </visual>
@@ -190,13 +190,13 @@
     <link name="rg2_r_moment_arm_link">
       <collision>
-        <origin xyz="0.0 0.0 0.0" rpy="0.0 0.0 0.0" />
-        <geometry>
-          <mesh filename="file://$(find ur_components_description)/meshes/onrobot/collision/RG2_RightMomentArm_col.STL" />
-        </geometry>
-      </collision>
-      <visual>
-        <origin xyz="0.00 0.00 0.00" rpy="0.00 0.00 0.00" />
-        <geometry>
-          <mesh filename="file://$(find ur_components_description)/meshes/onrobot/visual/RG2_RightMomentArm_vis.STL" />
+        <origin xyz="0.0 0.0 -0.02" rpy="${pi} 0.0 0.0" />
+        <geometry>
+          <mesh filename="file://$(find ur_components_description)/meshes/onrobot/moment_arm.stl" />
+        </geometry>
+      </collision>
+      <visual>
+        <origin xyz="0.0 0.0 -0.02" rpy="${pi} 0.0 0.0" />
+        <geometry>
+          <mesh filename="file://$(find ur_components_description)/meshes/onrobot/moment_arm.dae" />
         </geometry>
       </visual>
@@ -227,13 +227,13 @@
     <link name="rg2_r_finger_link">
       <collision>
-        <origin xyz="0.0 0.0 0.0" rpy="0.0 0.0 0.0" />
-        <geometry>
-          <mesh filename="file://$(find ur_components_description)/meshes/onrobot/collision/RG2_RightFinger_col.STL" />
-        </geometry>
-      </collision>
-      <visual>
-        <origin xyz="0.0 0.0 0.0" rpy="0.0 0.0 0.0" />
-        <geometry>
-          <mesh filename="file://$(find ur_components_description)/meshes/onrobot/visual/RG2_RightFinger_vis.STL" />
+        <origin xyz="0.0 0.0 -0.02" rpy="${pi} 0.0 0.0" />
+        <geometry>
+          <mesh filename="file://$(find ur_components_description)/meshes/onrobot/finger.stl" />
+        </geometry>
+      </collision>
+      <visual>
+        <origin xyz="0.0 0.0 -0.02" rpy="${pi} 0.0 0.0" />
+        <geometry>
+          <mesh filename="file://$(find ur_components_description)/meshes/onrobot/finger.dae" />
         </geometry>
       </visual>
@@ -264,13 +264,13 @@
     <link name="rg2_r_truss_arm_link">
       <collision>
-        <origin xyz="0.0 0.0 0.0" rpy="0.0 0.0 0.0" />
-        <geometry>
-          <mesh filename="file://$(find ur_components_description)/meshes/onrobot/collision/RG2_RightTrussArm_col.STL" />
-        </geometry>
-      </collision>
-      <visual>
-        <origin xyz="0.0 0.0 0.0" rpy="0.0 0.0 0.0" />
-        <geometry>
-          <mesh filename="file://$(find ur_components_description)/meshes/onrobot/visual/RG2_RightTrussArm_vis.STL" />
+        <origin xyz="0.0 0.0 -0.02" rpy="${pi} 0.0 0.0" />
+        <geometry>
+          <mesh filename="file://$(find ur_components_description)/meshes/onrobot/truss_arm.stl" />
+        </geometry>
+      </collision>
+      <visual>
+        <origin xyz="0.0 0.0 -0.02" rpy="${pi} 0.0 0.0" />
+        <geometry>
+          <mesh filename="file://$(find ur_components_description)/meshes/onrobot/truss_arm.dae" />
         </geometry>
       </visual>
@@ -286,5 +286,5 @@
       <plugin name="gazebo_ros_control" filename="libgazebo_ros_control.so">
         <robotNamespace>/rg2</robotNamespace>
-        <robotSimType>gazebo_ros_control/DefaultRobotHWSim</robotSimType>
+        <!-- <robotSimType>gazebo_ros_control/DefaultRobotHWSim</robotSimType> -->
       </plugin>
     </gazebo>
